File: processor_39F8497B/39F8497B.kicad_sch (KiCad schematic)
At the start: 72 parts, among them CN1 DIN41612_3x40, CN2 DIN41612_3x32, CN3 DIN41612_3x16, CN4 DIN41612_3x16, IC1 74LS32, IC10 ALS1805, IC11 74LS244, IC12 ALS641, IC13 25F8945, IC14 74LS157, IC15 74LS157, IC16 M5M5179P, IC17 74LS157, IC18 ALS641, IC19 ALS641, IC2 74LS00, IC20 74LS245, IC21 73X3718, IC22 ALS641, IC23 ALS641, IC24 74LS245, IC25 74LS244, IC26 74LS244, IC27 74LS245, IC28 74LS245, IC29 74LS244, IC3 74LS02, IC30 74LS244, IC31 74LS244, IC32 74LS245, IC33 74LS245, IC34 74LS245, IC36 74LS09, IC37 74LS245, IC38 74LS245, IC39 74LS245, IC4 28C256, IC41 74LS373, IC5 66X2711, IC6 74LS244, IC7 74LS244, IC8 74LS244, IC9 74LS244, X1 20AKSS9G

Commit message: Found old changes to the processor schematic, so that project is updated again (And thanks to KiCad's new UUIDs the diff is huge)
Connections:
- net GND: now also CN1.~ (C9), CN2.~ (C9), CN4.~ (C9), IC1.7 (GND), IC10.15 (GND), IC10.4, IC11.1 (OEa), IC11.10 (GND), IC11.19 (OEb), IC12.10 (GND), IC13.1, IC13.108, IC13.19, IC13.28, IC13.36, IC13.37, IC13.47, IC13.55, IC13.91, IC14.15 (E), IC14.8 (GND), IC15.15 (E), IC15.8 (GND), IC17.15 (E), IC17.8 (GND), IC18.1 (DIR), IC18.10 (GND), IC19.10 (GND), IC2.7 (GND), IC20.10 (GND), IC20.19 (CE), IC21.10, IC21.102, IC21.105, IC21.112, IC21.120, IC21.127, IC21.131, IC21.139, IC21.19, IC21.21, IC21.24, IC21.27, IC21.31, IC21.34, IC21.4, IC21.41, IC21.50, IC21.55, IC21.61, IC21.69, IC21.7, IC21.76, IC21.80, IC21.84, IC21.88, IC21.91, IC21.93, IC21.96, IC22.10 (GND), IC23.10 (GND), IC24.10 (GND), IC24.19 (CE), IC25.10 (GND), IC26.10 (GND), IC27.10 (GND), IC28.10 (GND), IC28.19 (CE), IC29.1 (OEa), IC29.10 (GND), IC29.19 (OEb), IC30.10 (GND), IC31.10 (GND), IC32.10 (GND), IC33.10 (GND), IC33.19 (CE), IC34.10 (GND), IC36.7 (GND), IC37.10 (GND), IC38.10 (GND), IC39.10 (GND), IC4.14 (GND), IC41.1 (OE), IC41.10 (GND), IC5.13, IC5.38, IC5.63, IC5.88, IC6.10 (GND), IC7.1 (OEa), IC7.10 (GND), IC7.19 (OEb), IC8.1 (OEa), IC8.10 (GND), IC8.19 (OEb), IC9.1 (OEa), IC9.10 (GND), IC9.19 (OEb), IR9.1 (common), JP1.2 (Pin_2)
- net ##192: now reaches IC2.5
- net ##192: now also IC13.95, IC21.70, IC29.17 (I3b), IC5.45
- net ##187: now reaches IC5.12
- net ##187: now also IC13.61, IC19.18 (B1), IC21.103, IC34.18 (B0), IC37.18 (B0), IR17.9 (R8)
- net ##160: now reaches IC5.39
- net ##160: now also IC13.42, IC21.104, IC23.17 (B2), IC32.17 (B1), IC38.17 (B1), IR18.5 (R4)
- net ##195: now reaches IC5.41
- net ##195: now also IC13.94, IC21.62, IC29.11 (I0b)
- net ##186: now reaches IC5.42
- net ##186: now also IC13.60, IC19.17 (B2), IC21.29, IC34.17 (B1), IC37.17 (B1), IR17.10 (R9)
- net ##161: now reaches IC5.44
- net ##161: now also IC13.41, IC21.101, IC23.18 (B1), IC32.18 (B0), IC38.18 (B0), IR18.4 (R3)
- net ##194: now reaches IC5.46
- net ##194: now also IC10.18, IC10.7, IC21.63, IC29.13 (I1b)
- net ##155: now reaches IC5.56
- net ##155: now also IC13.48, IC21.106, IC23.12 (B7), IC32.12 (B6), IC38.12 (B6), IR18.10 (R9)
- net ##158: now reaches IC5.62
- net ##158: now also IC13.44, IC21.6, IC23.15 (B4), IC32.15 (B3), IC38.15 (B3), IR18.7 (R6)
- net ##159: now reaches IC5.64
- net ##159: now also IC13.43, IC21.8, IC23.16 (B3), IC32.16 (B2), IC38.16 (B2), IR18.6 (R5)
- net ##156: now reaches IC5.7
- net ##156: now also IC13.46, IC21.3, IC23.13 (B6), IC32.13 (B5), IC38.13 (B5), IR18.9 (R8)
- net ##154: now reaches IC5.72
- net ##154: now also IC13.49, IC21.5, IC23.11 (B8), IC32.11 (B7), IC38.11 (B7), IR18.3 (R2)
- net ##157: now reaches IC5.81
- net ##157: now also IC13.45, IC21.98, IC23.14 (B5), IC32.14 (B4), IC38.14 (B4), IR18.8 (R7)
- net ##146: now reaches IR5.10 (R9)
- net ##146: now also CN2.~ (C9), IC13.35
- net ##151: now reaches IR5.3 (R2)
- net ##151: now also CN2.~ (A9), CN?.~ (A9), IC13.31
- net ##153: now reaches IR5.4 (R3)
- net ##153: now also CN2.~ (B9), IC13.30
- net ##152: now reaches IR5.5 (R4)
- net ##152: now also CN2.~ (C9), IC13.29
- net ##148: now reaches IR5.6 (R5)
- net ##148: now also CN2.~ (A9), CN?.~ (A9), IC13.34
- net ##149: now reaches IR5.7 (R6)
- net ##149: now also CN2.~ (B9), IC13.33
- net ##150: now reaches IR5.8 (R7)
- net ##150: now also CN2.~ (C9), IC13.32
- net ##147: now reaches IR5.9 (R8)
- net ##147: now also CN2.~ (B9), IC13.40
- net ##139: now reaches IR6.10 (R9)
- net ##139: now also CN2.~ (B9), IC13.24
- net ##141: now reaches IR6.3 (R2)
- net ##141: now also CN2.~ (C9), IC13.26
- net ##138: now reaches IR6.4 (R3)
- net ##138: now also CN2.~ (B9), IC13.27
- net ##142: now reaches IR6.5 (R4)
- net ##142: now also CN2.~ (C9), IC13.23
- net ##145: now reaches IR6.6 (R5)
- net ##145: now also CN2.~ (A9), CN?.~ (A9), IC13.22
- net ##140: now reaches IR6.7 (R6)
- net ##140: now also CN2.~ (B9), IC13.21
- net ##143: now reaches IR6.8 (R7)
- net ##143: now also CN2.~ (C9), IC13.20
- net ##144: now reaches IR6.9 (R8)
- net ##144: now also CN2.~ (A9), CN?.~ (A9), IC13.25
- net ##126: now reaches IC13.10
- net ##126: now also IC14.6 (I1b)
- net ##127: now reaches IC13.11
- net ##127: now also IC14.3 (I1a)
- net ##197: now reaches IC13.118
- net ##197: now also IC29.6 (I2a)
- net ##196: now reaches IC13.119
- net ##196: now also IC29.8 (I3a)
- net ##120: now reaches IC13.4
- net ##120: now also IC15.13 (I1d)
- net ##121: now reaches IC13.5
- net ##121: now also IC15.10 (I1c)
- net ##122: now reaches IC13.6
- net ##122: now also IC15.6 (I1b)
- net ##123: now reaches IC13.7
- net ##123: now also IC15.3 (I1a)
- net ##193: now reaches IC13.73
- net ##193: now also IC20.1 (A->B), IC21.144, IC24.1 (A->B), IC28.1 (A->B), IC29.15 (I2b), IC33.1 (A->B)
- net ##124: now reaches IC13.8
- net ##124: now also IC14.13 (I1d)
- net ##125: now reaches IC13.9
- net ##125: now also IC14.10 (I1c)
- net ##167: now reaches IR14.10 (R9)
- net ##167: now also CN1.~ (B9), IC23.4 (A3)
- net ##162: now reaches IR14.3 (R2)
- net ##162: now also CN1.~ (B9), IC23.9 (A8)
- net ##163: now reaches IR14.4 (R3)
- net ##163: now also CN1.~ (A9), IC23.8 (A7)
- net ##164: now reaches IR14.5 (R4)
- net ##164: now also CN1.~ (A9), IC23.7 (A6)
- net ##165: now reaches IR14.6 (R5)
- net ##165: now also CN1.~ (B9), IC23.6 (A5)
- net ##166: now reaches IR14.7 (R6)
- net ##166: now also CN1.~ (C9), IC23.5 (A4)
- net ##168: now reaches IR14.8 (R7)
- net ##168: now also CN1.~ (B9), IC23.3 (A2)
- net ##169: now reaches IR14.9 (R8)
- net ##169: now also CN1.~ (C9), IC23.2 (A1)
- net ##188: now reaches IR19.10 (R9)
- net ##188: now also CN1.~ (C9), IC34.3 (A1)
- net ##189: now reaches IR19.9 (R8)
- net ##189: now also CN1.~ (B9), IC34.2 (A0)
- net ##185: now reaches CN3.~ (A9)
- net ##185: now also IC32.2 (A0)
- net ##182: now reaches CN3.~ (B9)
- net ##182: now also IC32.5 (A3)
- net ##134: now reaches IC14.12 (Zd)
- net ##134: now also CN2.~ (B9)
- net ##137: now reaches IC14.4 (Za)
- net ##137: now also CN2.~ (B9)
- net ##136: now reaches IC14.7 (Zb)
- net ##136: now also CN2.~ (C9)
- net ##135: now reaches IC14.9 (Zc)
- net ##135: now also CN2.~ (B9)
- net ##130: now reaches IC15.12 (Zd)
- net ##130: now also CN2.~ (A9), CN?.~ (A9)
- net ##133: now reaches IC15.4 (Za)
- net ##133: now also CN2.~ (B9)
- net ##132: now reaches IC15.7 (Zb)
- net ##132: now also CN2.~ (B9)
- net ##131: now reaches IC15.9 (Zc)
- net ##131: now also CN2.~ (A9), CN?.~ (A9)
- net ##129: now reaches IC17.4 (Za)
- net ##129: now also CN2.~ (C9)
- net ##128: now reaches IC17.7 (Zb)
- net ##128: now also CN2.~ (C9)
- net ##198: now reaches IC21.67
- net ##198: now also IC29.4 (I1a)
- net ##199: now reaches IC21.74
- net ##199: now also IC29.2 (I0a)
- net ##177: now reaches IC27.2 (A0)
- net ##177: now also CN3.~ (A9)
- net ##176: now reaches IC27.3 (A1)
- net ##176: now also CN3.~ (A9)
- net ##175: now reaches IC27.4 (A2)
- net ##175: now also CN3.~ (A9)
- net ##174: now reaches IC27.5 (A3)
- net ##174: now also CN3.~ (B9)
- net ##173: now reaches IC27.6 (A4)
- net ##173: now also CN3.~ (B9)
- net ##172: now reaches IC27.7 (A5)
- net ##172: now also CN3.~ (B9)
- net ##171: now reaches IC27.8 (A6)
- net ##171: now also CN3.~ (C9)
- net ##170: now reaches IC27.9 (A7)
- net ##170: now also CN3.~ (C9)
- net ##184: now reaches IC32.3 (A1)
- net ##184: now also CN3.~ (A9)
- net ##183: now reaches IC32.4 (A2)
- net ##183: now also CN3.~ (A9)
- net ##181: now reaches IC32.6 (A4)
- net ##181: now also CN3.~ (B9)
- net ##180: now reaches IC32.7 (A5)
- net ##180: now also CN3.~ (B9)
- net ##179: now reaches IC32.8 (A6)
- net ##179: now also CN3.~ (C9)
- net ##178: now reaches IC32.9 (A7)
- net ##178: now also CN3.~ (C9)
- net ##191: now reaches IC37.2 (A0)
- net ##191: now also CN3.~ (C9)
- net ##190: now reaches IC37.3 (A1)
- net ##190: now also CN3.~ (C9)
- new net: CN2.~ (A9), CN?.~ (A9) (x22)
- no-connect marks 35 -> 71
Other:
- moved on the sheet: IR5, IR6
